Commit message: Project 4 - mapping.launch errors

File: my_robot/urdf/my_robot.xacro (robot description, xacro)
@@ -145,4 +145,5 @@
     </visual>
   </link>
+  <!-- ****************************************************************** -->
 <joint type="fixed" name="camera_joint">
     <origin xyz="0.2 0 0" rpy="0 0 0"/>
@@ -153,4 +154,12 @@
     <dynamics damping="1.0" friction="1.0"/>
   </joint>
+<joint name="camera_optical_joint" type="fixed">
+  <origin xyz="0 0 0" rpy="-1.5707 0 -1.5707"/>
+  <parent link="camera_link"/>
+  <child link="camera_link_optical"/>
+</joint>
+<link name="camera_link_optical">
+</link>
+<!-- ****************************************************************** -->
 <link name='hokuyo'>
  <pose>0 0 0.1 0 0 0</pose>

Commit message: P4

File: my_robot/urdf/my_robot.xacro (robot description, xacro)
@@ -156,5 +156,5 @@
 <joint name="camera_optical_joint" type="fixed">
   <origin xyz="0 0 0" rpy="-1.5707 0 -1.5707"/>
-  <parent link="camera_link"/>
+  <parent link="camera"/> <!-- ******-->
   <child link="camera_link_optical"/>
 </joint>
